Commit message: added navigation and changed robot to skid steer

File: src/koala_description/urdf/macros.xacro (robot description, xacro)
@@ -49,7 +49,7 @@
     </gazebo>
     <joint name="${lr}_wheel_hinge" type="continuous">
-      <parent link="chassis"/>
+      <parent link="body"/>
       <child link="${lr}_wheel"/>
-    <origin xyz="${-wheelPos+chassisLength/2} ${tY*wheelWidth/2+tY*chassisWidth/2} ${wheelRadius}" rpy="0 0 0" />
+    <origin xyz="${-wheelPos+bodyLength/2} ${tY*wheelWidth/2+tY*bodyWidth/2} ${wheelRadius}" rpy="0 0 0" />
       <axis xyz="0 1 0" rpy="0 0 0" />
       <limit effort="10000" velocity="10000"/>
