Commit message: add 16 IR sensors

File: src/koala_description/urdf/koala.xacro (robot description, xacro)
@@ -31,4 +31,5 @@
     </visual>
   </link>
+<!--3x2 wheels skid steer robot-->>
   <link name="left_wheel_middle">
     <!--origin xyz="0.1 0.13 0.1" rpy="0 1.5707 1.5707"/-->
@@ -229,5 +230,5 @@
     <joint_properties damping="0.0" friction="0.0"/>
   </joint>
-  <!-- Camera -->
+<!-- Camera -->
  <link name="camera">
     <collision>
@@ -257,3 +258,409 @@
     <child link="camera"/>
   </joint>
+<!--IR sensors right front-->
+  <joint name="ir_r0_joint" type="fixed">
+    <axis xyz="0 1 0" />
+    <origin rpy="0 0 0" xyz="0.325 -0.03 0.05" />
+    <parent link="body"/>
+    <child link="ir_r0"/>
+  </joint>
+  <link name="ir_r0">
+    <collision>
+      <origin xyz="0 0 0" rpy="0 0 0"/>
+      <geometry>
+        <box size="0.01 0.01 0.01"/>
+      </geometry>
+    </collision>
+    <visual>
+      <origin xyz="0 0 0" rpy="0 0 0"/>
+      <geometry>
+        <box size="0.01 0.01 0.01"/>
+      </geometry>
+    </visual>
+    <inertial>
+      <mass value="1e-5" />
+      <origin xyz="0 0 0" rpy="0 0 0"/>
+      <inertia ixx="1e-6" ixy="0" ixz="0" iyy="1e-6" iyz="0" izz="1e-6" />
+    </inertial>
+  </link>
+  <joint name="ir_r1_joint" type="fixed">
+    <axis xyz="0 1 0" />
+    <origin rpy="0 0 -0.1" xyz="0.3245 -0.07 0.05" />
+    <parent link="body"/>
+    <child link="ir_r1"/>
+  </joint>
+  <link name="ir_r1">
+    <collision>
+      <origin xyz="0 0 0" rpy="0 0 0"/>
+      <geometry>
+        <box size="0.01 0.01 0.01"/>
+      </geometry>
+    </collision>
+    <visual>
+      <origin xyz="0 0 0" rpy="0 0 0"/>
+      <geometry>
+        <box size="0.01 0.01 0.01"/>
+      </geometry>
+    </visual>
+    <inertial>
+      <mass value="1e-5" />
+      <origin xyz="0 0 0" rpy="0 0 0"/>
+      <inertia ixx="1e-6" ixy="0" ixz="0" iyy="1e-6" iyz="0" izz="1e-6" />
+    </inertial>
+  </link>
+  <joint name="ir_r2_joint" type="fixed">
+    <axis xyz="0 1 0" />
+    <origin rpy="0 0 -0.3" xyz="0.324 -0.12 0.05" />
+    <parent link="body"/>
+    <child link="ir_r2"/>
+  </joint>
+  <link name="ir_r2">
+    <collision>
+      <origin xyz="0 0 0" rpy="0 0 0"/>
+      <geometry>
+        <box size="0.01 0.01 0.01"/>
+      </geometry>
+    </collision>
+    <visual>
+      <origin xyz="0 0 0" rpy="0 0 0"/>
+      <geometry>
+        <box size="0.01 0.01 0.01"/>
+      </geometry>
+    </visual>
+    <inertial>
+      <mass value="1e-5" />
+      <origin xyz="0 0 0" rpy="0 0 0"/>
+      <inertia ixx="1e-6" ixy="0" ixz="0" iyy="1e-6" iyz="0" izz="1e-6" />
+    </inertial>
+  </link>
+  <joint name="ir_r3_joint" type="fixed">
+    <axis xyz="0 1 0" />
+    <origin rpy="0 0 -0.7" xyz="0.323 -0.17 0.05" />
+    <parent link="body"/>
+    <child link="ir_r3"/>
+  </joint>
+  <link name="ir_r3">
+    <collision>
+      <origin xyz="0 0 0" rpy="0 0 0"/>
+      <geometry>
+        <box size="0.01 0.01 0.01"/>
+      </geometry>
+    </collision>
+    <visual>
+      <origin xyz="0 0 0" rpy="0 0 0"/>
+      <geometry>
+        <box size="0.01 0.01 0.01"/>
+      </geometry>
+    </visual>
+    <inertial>
+      <mass value="1e-5" />
+      <origin xyz="0 0 0" rpy="0 0 0"/>
+      <inertia ixx="1e-6" ixy="0" ixz="0" iyy="1e-6" iyz="0" izz="1e-6" />
+    </inertial>
+  </link>
+<!--IR sensors right-->
+  <joint name="ir_r4_joint" type="fixed">
+    <axis xyz="0 1 0" />
+    <origin rpy="0 0 -1.6" xyz="0.1 -0.175 0.05" />
+    <parent link="body"/>
+    <child link="ir_r4"/>
+  </joint>
+  <link name="ir_r4">
+    <collision>
+      <origin xyz="0 0 0" rpy="0 0 0"/>
+      <geometry>
+        <box size="0.01 0.01 0.01"/>
+      </geometry>
+    </collision>
+    <visual>
+      <origin xyz="0 0 0" rpy="0 0 0"/>
+      <geometry>
+        <box size="0.01 0.01 0.01"/>
+      </geometry>
+    </visual>
+    <inertial>
+      <mass value="1e-5" />
+      <origin xyz="0 0 0" rpy="0 0 0"/>
+      <inertia ixx="1e-6" ixy="0" ixz="0" iyy="1e-6" iyz="0" izz="1e-6" />
+    </inertial>
+  </link>
+  <joint name="ir_r5_joint" type="fixed">
+    <axis xyz="0 1 0" />
+    <origin rpy="0 0 -1.6" xyz="-0.1 -0.175 0.05" />
+    <parent link="body"/>
+    <child link="ir_r5"/>
+  </joint>
+  <link name="ir_r5">
+    <collision>
+      <origin xyz="0 0 0" rpy="0 0 0"/>
+      <geometry>
+        <box size="0.01 0.01 0.01"/>
+      </geometry>
+    </collision>
+    <visual>
+      <origin xyz="0 0 0" rpy="0 0 0"/>
+      <geometry>
+        <box size="0.01 0.01 0.01"/>
+      </geometry>
+    </visual>
+    <inertial>
+      <mass value="1e-5" />
+      <origin xyz="0 0 0" rpy="0 0 0"/>
+      <inertia ixx="1e-6" ixy="0" ixz="0" iyy="1e-6" iyz="0" izz="1e-6" />
+    </inertial>
+  </link>
+<!--IR sensors right rear-->
+  <joint name="ir_r6_joint" type="fixed">
+    <axis xyz="0 1 0" />
+    <origin rpy="0 0 -2.4" xyz="-0.325 -0.17 0.05" />
+    <parent link="body"/>
+    <child link="ir_r6"/>
+  </joint>
+  <link name="ir_r6">
+    <collision>
+      <origin xyz="0 0 0" rpy="0 0 0"/>
+      <geometry>
+        <box size="0.01 0.01 0.01"/>
+      </geometry>
+    </collision>
+    <visual>
+      <origin xyz="0 0 0" rpy="0 0 0"/>
+      <geometry>
+        <box size="0.01 0.01 0.01"/>
+      </geometry>
+    </visual>
+    <inertial>
+      <mass value="1e-5" />
+      <origin xyz="0 0 0" rpy="0 0 0"/>
+      <inertia ixx="1e-6" ixy="0" ixz="0" iyy="1e-6" iyz="0" izz="1e-6" />
+    </inertial>
+  </link>
+  <joint name="ir_r7_joint" type="fixed">
+    <axis xyz="0 1 0" />
+    <origin rpy="0 0 -3.1" xyz="-0.325 -0.05 0.05" />
+    <parent link="body"/>
+    <child link="ir_r7"/>
+  </joint>
+  <link name="ir_r7">
+    <collision>
+      <origin xyz="0 0 0" rpy="0 0 0"/>
+      <geometry>
+        <box size="0.01 0.01 0.01"/>
+      </geometry>
+    </collision>
+    <visual>
+      <origin xyz="0 0 0" rpy="0 0 0"/>
+      <geometry>
+        <box size="0.01 0.01 0.01"/>
+      </geometry>
+    </visual>
+    <inertial>
+      <mass value="1e-5" />
+      <origin xyz="0 0 0" rpy="0 0 0"/>
+      <inertia ixx="1e-6" ixy="0" ixz="0" iyy="1e-6" iyz="0" izz="1e-6" />
+    </inertial>
+  </link>
+<!--IR sensors left front-->
+  <joint name="ir_l0_joint" type="fixed">
+    <axis xyz="0 1 0" />
+    <origin rpy="0 0 0" xyz="0.325 0.03 0.05" />
+    <parent link="body"/>
+    <child link="ir_l0"/>
+  </joint>
+  <link name="ir_l0">
+    <collision>
+      <origin xyz="0 0 0" rpy="0 0 0"/>
+      <geometry>
+        <box size="0.01 0.01 0.01"/>
+      </geometry>
+    </collision>
+    <visual>
+      <origin xyz="0 0 0" rpy="0 0 0"/>
+      <geometry>
+        <box size="0.01 0.01 0.01"/>
+      </geometry>
+    </visual>
+    <inertial>
+      <mass value="1e-5" />
+      <origin xyz="0 0 0" rpy="0 0 0"/>
+      <inertia ixx="1e-6" ixy="0" ixz="0" iyy="1e-6" iyz="0" izz="1e-6" />
+    </inertial>
+  </link>
+  <joint name="ir_l1_joint" type="fixed">
+    <axis xyz="0 1 0" />
+    <origin rpy="0 0 0.1" xyz="0.3245 0.07 0.05" />
+    <parent link="body"/>
+    <child link="ir_l1"/>
+  </joint>
+  <link name="ir_l1">
+    <collision>
+      <origin xyz="0 0 0" rpy="0 0 0"/>
+      <geometry>
+        <box size="0.01 0.01 0.01"/>
+      </geometry>
+    </collision>
+    <visual>
+      <origin xyz="0 0 0" rpy="0 0 0"/>
+      <geometry>
+        <box size="0.01 0.01 0.01"/>
+      </geometry>
+    </visual>
+    <inertial>
+      <mass value="1e-5" />
+      <origin xyz="0 0 0" rpy="0 0 0"/>
+      <inertia ixx="1e-6" ixy="0" ixz="0" iyy="1e-6" iyz="0" izz="1e-6" />
+    </inertial>
+  </link>
+  <joint name="ir_l2joint" type="fixed">
+    <axis xyz="0 1 0" />
+    <origin rpy="0 0 0.3" xyz="0.324 0.12 0.05" />
+    <parent link="body"/>
+    <child link="ir_l2"/>
+  </joint>
+  <link name="ir_l2">
+    <collision>
+      <origin xyz="0 0 0" rpy="0 0 0"/>
+      <geometry>
+        <box size="0.01 0.01 0.01"/>
+      </geometry>
+    </collision>
+    <visual>
+      <origin xyz="0 0 0" rpy="0 0 0"/>
+      <geometry>
+        <box size="0.01 0.01 0.01"/>
+      </geometry>
+    </visual>
+    <inertial>
+      <mass value="1e-5" />
+      <origin xyz="0 0 0" rpy="0 0 0"/>
+      <inertia ixx="1e-6" ixy="0" ixz="0" iyy="1e-6" iyz="0" izz="1e-6" />
+    </inertial>
+  </link>
+  <joint name="ir_l3_joint" type="fixed">
+    <axis xyz="0 1 0" />
+    <origin rpy="0 0 0.7" xyz="0.323 0.17 0.05" />
+    <parent link="body"/>
+    <child link="ir_l3"/>
+  </joint>
+  <link name="ir_l3">
+    <collision>
+      <origin xyz="0 0 0" rpy="0 0 0"/>
+      <geometry>
+        <box size="0.01 0.01 0.01"/>
+      </geometry>
+    </collision>
+    <visual>
+      <origin xyz="0 0 0" rpy="0 0 0"/>
+      <geometry>
+        <box size="0.01 0.01 0.01"/>
+      </geometry>
+    </visual>
+    <inertial>
+      <mass value="1e-5" />
+      <origin xyz="0 0 0" rpy="0 0 0"/>
+      <inertia ixx="1e-6" ixy="0" ixz="0" iyy="1e-6" iyz="0" izz="1e-6" />
+    </inertial>
+  </link>
+<!--IR sensors left-->
+  <joint name="ir_l4_joint" type="fixed">
+    <axis xyz="0 1 0" />
+    <origin rpy="0 0 1.6" xyz="0.1 0.175 0.05" />
+    <parent link="body"/>
+    <child link="ir_l4"/>
+  </joint>
+  <link name="ir_l4">
+    <collision>
+      <origin xyz="0 0 0" rpy="0 0 0"/>
+      <geometry>
+        <box size="0.01 0.01 0.01"/>
+      </geometry>
+    </collision>
+    <visual>
+      <origin xyz="0 0 0" rpy="0 0 0"/>
+      <geometry>
+        <box size="0.01 0.01 0.01"/>
+      </geometry>
+    </visual>
+    <inertial>
+      <mass value="1e-5" />
+      <origin xyz="0 0 0" rpy="0 0 0"/>
+      <inertia ixx="1e-6" ixy="0" ixz="0" iyy="1e-6" iyz="0" izz="1e-6" />
+    </inertial>
+  </link>
+  <joint name="ir_l5_joint" type="fixed">
+    <axis xyz="0 1 0" />
+    <origin rpy="0 0 1.6" xyz="-0.1 0.175 0.05" />
+    <parent link="body"/>
+    <child link="ir_l5"/>
+  </joint>
+  <link name="ir_l5">
+    <collision>
+      <origin xyz="0 0 0" rpy="0 0 0"/>
+      <geometry>
+        <box size="0.01 0.01 0.01"/>
+      </geometry>
+    </collision>
+    <visual>
+      <origin xyz="0 0 0" rpy="0 0 0"/>
+      <geometry>
+        <box size="0.01 0.01 0.01"/>
+      </geometry>
+    </visual>
+    <inertial>
+      <mass value="1e-5" />
+      <origin xyz="0 0 0" rpy="0 0 0"/>
+      <inertia ixx="1e-6" ixy="0" ixz="0" iyy="1e-6" iyz="0" izz="1e-6" />
+    </inertial>
+  </link>
+<!--IR sensors left rear-->
+  <joint name="ir_l6_joint" type="fixed">
+    <axis xyz="0 1 0" />
+    <origin rpy="0 0 2.4" xyz="-0.325 0.17 0.05" />
+    <parent link="body"/>
+    <child link="ir_l6"/>
+  </joint>
+  <link name="ir_l6">
+    <collision>
+      <origin xyz="0 0 0" rpy="0 0 0"/>
+      <geometry>
+        <box size="0.01 0.01 0.01"/>
+      </geometry>
+    </collision>
+    <visual>
+      <origin xyz="0 0 0" rpy="0 0 0"/>
+      <geometry>
+        <box size="0.01 0.01 0.01"/>
+      </geometry>
+    </visual>
+    <inertial>
+      <mass value="1e-5" />
+      <origin xyz="0 0 0" rpy="0 0 0"/>
+      <inertia ixx="1e-6" ixy="0" ixz="0" iyy="1e-6" iyz="0" izz="1e-6" />
+    </inertial>
+  </link>
+  <joint name="ir_l7_joint" type="fixed">
+    <axis xyz="0 1 0" />
+    <origin rpy="0 0 3.1" xyz="-0.325 0.05 0.05" />
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
Commit message: added kinect sensor

File: src/koala_description/urdf/koala.xacro (robot description, xacro)
@@ -231,30 +231,28 @@
   </joint>
 <!-- Camera -->
- <link name="camera">
-    <collision>
-      <origin xyz="0 0 0" rpy="0 0 0"/>
-      <geometry>
-        <box size="${cameraSize} ${cameraSize} ${cameraSize}"/>
-      </geometry>
-    </collision>
-    <visual>
-      <origin xyz="0 0 0" rpy="0 0 0"/>
-      <geometry>
-        <box size="${cameraSize} ${cameraSize} ${cameraSize}"/>
-      </geometry>
-      <material name="black"/>
-    </visual>
-    <inertial>
-      <mass value="${cameraMass}" />
-      <origin xyz="0 0 0" rpy="0 0 0"/>
-      <box_inertia m="${cameraMass}" x="${cameraSize}" y="${cameraSize}" z="${cameraSize}" />
-      <inertia ixx="1e-6" ixy="0" ixz="0" iyy="1e-6" iyz="0" izz="1e-6" />
-    </inertial>
-  </link>
-  <joint name="camera_joint" type="fixed">
-    <axis xyz="0 1 0" />
-    <origin xyz="0.3 0.0 0.1" rpy="0 0 0"/>
-    <parent link="body"/>
-    <child link="camera"/>
+  <link name="kinect">
+    <collision name="collision">
+      <origin xyz="0 0 0" rpy="0 0 0"/>
+      <geometry>
+        <box size="0.073000 0.276000 0.072000"/>
+      </geometry>
+    </collision>
+    <visual name="visual">
+      <origin xyz="0 0 0" rpy="0 0 0"/>
+      <geometry>
+        <mesh filename="package://koala_description/meshes/kinect.dae"/>
+      </geometry>
+    </visual>
+    <inertial>
+      <mass value="1e-5" />
+      <origin xyz="0 0 0" rpy="0 0 0"/>
+      <inertia ixx="1e-6" ixy="0" ixz="0" iyy="1e-6" iyz="0" izz="1e-6" />
+    </inertial>
+  </link>
+  <joint name="kinect_joint" type="fixed">
+    <axis xyz="0 1 0" />
+    <origin xyz="0.28 0.0 0.11" rpy="0 0 1.57"/>
+    <parent link="body"/>
+    <child link="kinect"/>
   </joint>
 <!--IR sensors right front-->

Commit message: fix kinect pointing wrong direction

File: src/koala_description/urdf/koala.xacro (robot description, xacro)
@@ -233,5 +233,5 @@
   <link name="kinect">
     <collision name="collision">
-      <origin xyz="0 0 0" rpy="0 0 0"/>
+      <origin xyz="0 0 0" rpy="0 0 1.57"/>
       <geometry>
         <box size="0.073000 0.276000 0.072000"/>
@@ -239,5 +239,5 @@
     </collision>
     <visual name="visual">
-      <origin xyz="0 0 0" rpy="0 0 0"/>
+      <origin xyz="0 0 0" rpy="0 0 1.57"/>
       <geometry>
         <mesh filename="package://koala_description/meshes/kinect.dae"/>
@@ -252,8 +252,22 @@
   <joint name="kinect_joint" type="fixed">
     <axis xyz="0 1 0" />
-    <origin xyz="0.28 0.0 0.11" rpy="0 0 1.57"/>
+    <origin xyz="0.28 0.0 0.11" rpy="0 0 0"/>
     <parent link="body"/>
     <child link="kinect"/>
   </joint>
+<!-- generate an optical frame
+      http://www.ros.org/reps/rep-0103.html#suffix-frames
+      so that ros and opencv can operate on the camera frame correctly
+      -->
+  <joint name="kinect_optical_joint" type="fixed">
+    <!-- these values have to be these values otherwise the gazebo camera
+        image won't be aligned properly with the frame it is supposedly
+        originating from -->
+    <origin xyz="0 0 0" rpy="-1.57 0 -1.57"/>
+    <parent link="kinect"/>
+    <child link="kinect_link_optical"/>
+  </joint>
+  <link name="kinect_link_optical">
+  </link>
 <!--IR sensors right front-->
   <joint name="ir_r0_joint" type="fixed">

Commit message: add color to ir visualize false

File: src/koala_description/urdf/koala.xacro (robot description, xacro)
@@ -289,4 +289,5 @@
         <box size="0.01 0.01 0.01"/>
       </geometry>
+      <material name="black"/>
     </visual>
     <inertial>
@@ -314,4 +315,5 @@
         <box size="0.01 0.01 0.01"/>
       </geometry>
+      <material name="black"/>
     </visual>
     <inertial>
@@ -339,4 +341,5 @@
         <box size="0.01 0.01 0.01"/>
       </geometry>
+      <material name="black"/>
     </visual>
     <inertial>
@@ -364,4 +367,5 @@
         <box size="0.01 0.01 0.01"/>
       </geometry>
+      <material name="black"/>
     </visual>
     <inertial>
@@ -390,4 +394,5 @@
         <box size="0.01 0.01 0.01"/>
       </geometry>
+      <material name="black"/>
     </visual>
     <inertial>
@@ -415,4 +420,5 @@
         <box size="0.01 0.01 0.01"/>
       </geometry>
+      <material name="black"/>
     </visual>
     <inertial>
@@ -441,4 +447,5 @@
         <box size="0.01 0.01 0.01"/>
       </geometry>
+      <material name="black"/>
     </visual>
     <inertial>
@@ -466,4 +473,5 @@
         <box size="0.01 0.01 0.01"/>
       </geometry>
+      <material name="black"/>
     </visual>
     <inertial>
@@ -492,4 +500,5 @@
         <box size="0.01 0.01 0.01"/>
       </geometry>
+      <material name="black"/>
     </visual>
     <inertial>
@@ -517,4 +526,5 @@
         <box size="0.01 0.01 0.01"/>
       </geometry>
+      <material name="black"/>
     </visual>
     <inertial>
@@ -542,4 +552,5 @@
         <box size="0.01 0.01 0.01"/>
       </geometry>
+      <material name="black"/>
     </visual>
     <inertial>
@@ -567,4 +578,5 @@
         <box size="0.01 0.01 0.01"/>
       </geometry>
+      <material name="black"/>
     </visual>
     <inertial>
@@ -593,4 +605,5 @@
         <box size="0.01 0.01 0.01"/>
       </geometry>
+      <material name="black"/>
     </visual>
     <inertial>
@@ -618,4 +631,5 @@
         <box size="0.01 0.01 0.01"/>
       </geometry>
+      <material name="black"/>
     </visual>
     <inertial>
@@ -644,4 +658,5 @@
         <box size="0.01 0.01 0.01"/>
       </geometry>
+      <material name="black"/>
     </visual>
     <inertial>
@@ -669,4 +684,5 @@
         <box size="0.01 0.01 0.01"/>
       </geometry>
+      <material name="black"/>
     </visual>
     <inertial>
